Commit message: working

File: go2_robot_sdk/urdf/go2.urdf (robot description, URDF)
Before this commit: robot go2, 33 links, 32 joints
Links:
- removed link radar
- added link LIDAR, mass 0
Joints:
- removed joint radar_joint
- added joint LIDAR_joint: type fixed, parent base_link, child LIDAR, origin xyz=0.28945 0 -0.046825 rpy=0 2.8782 0, axis 0 0 0

Commit message: Update go2.urdf

File: go2_robot_sdk/urdf/go2.urdf (robot description, URDF)
Before this commit: robot Go2, 33 links, 32 joints
Joints:
- removed joint base_footprint_joint
- added joint base_link_joint: type fixed, parent base_link, child base_footprint, origin xyz=0 0 0 rpy=0 0 0

Commit message: EKF optimisation

File: go2_robot_sdk/urdf/go2.urdf (robot description, URDF)
Before this commit: robot Go2, 33 links, 32 joints
Links:
- removed link imu
- added link GPS, mass 0; visual cylinder length=0.03 radius=0.03
- added link IMU, mass 0
Joints:
- removed joint imu_joint
- added joint GPS_joint: type fixed, parent base_link, child GPS, origin xyz=0.22 0 0.12 rpy=0 0 0, axis 0 0 0
- added joint IMU_joint: type fixed, parent base_link, child IMU, origin xyz=-0.02557 0 0.04232 rpy=0 0 0, axis 0 0 0

Commit message: align witmotion to unitree

File: go2_robot_sdk/urdf/go2.urdf (robot description, URDF)
Before this commit: robot Go2, 34 links, 33 joints
Links:
- added link IMU_wit, mass 0; visual cylinder length=0.02 radius=0.02
- link GPS: geometry visual cylinder length=0.02 radius=0.03
Joints:
- added joint IMU_joint_wit: type fixed, parent base_link, child IMU_wit, origin xyz=0.22 0 0.10 rpy=0 0 0, axis 0 0 0
